File: learnings/MPPT/mppt.kicad_sch (KiCad schematic)
At the start: 20 parts

Commit message: MPPT_v2 working
Parts:
- removed V3: i(Vipv1), symbol Simulation_SPICE:VDC
- added Bsense1: BSOURCE, symbol Simulation_SPICE:BSOURCE
Connections:
- net 0: now also Bsense1.2 (N-)
- net a: now reaches filtfast1.1 (in), filtslow1.1 (in), mul1.3
- net at mul1.2: now also Bsense1.1 (N+)
Other:
- moved on the sheet: mul1
